File: KiCAD/TrackingGenerator.kicad_sch (KiCad schematic)
At the start: 65 parts, among them IC1 ABA-52563-BLKG, IC2 ABA-52563-BLKG, IC3 ABA-52563-BLKG, J1 Conn_Coaxial, J2 Conn_Coaxial, J3 Screw_Terminal_01x02, J4 Conn_Coaxial, M1 PAM-42, U1 L7805

Commit message: More routing work
Parts:
- J1, J2, J4: footprint Connector_Coaxial:SMA_Amphenol_132134-10_Vertical -> Connector_Coaxial:SMA_Amphenol_132289_EdgeMount
Changed lines of the file:
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@@
       (effects (font (size 1.27 1.27)) (justify left))
     )
-    (property "Footprint" "Connector_Coaxial:SMA_Amphenol_132134-10_Vertical" (id 2) (at 41.91 57.15 0)
+    (property "Footprint" "Connector_Coaxial:SMA_Amphenol_132289_EdgeMount" (id 2) (at 41.91 57.15 0)
       (effects (font (size 1.27 1.27)) hide)
     )
@@
       (effects (font (size 1.27 1.27)) (justify left))
     )
-    (property "Footprint" "Connector_Coaxial:SMA_Amphenol_132134-10_Vertical" (id 2) (at 276.86 100.33 0)
+    (property "Footprint" "Connector_Coaxial:SMA_Amphenol_132289_EdgeMount" (id 2) (at 276.86 100.33 0)
       (effects (font (size 1.27 1.27)) hide)
     )
@@
       (effects (font (size 1.27 1.27)) (justify left))
     )
-    (property "Footprint" "Connector_Coaxial:SMA_Amphenol_132134-10_Vertical" (id 2) (at 41.91 111.76 0)
+    (property "Footprint" "Connector_Coaxial:SMA_Amphenol_132289_EdgeMount" (id 2) (at 41.91 111.76 0)
       (effects (font (size 1.27 1.27)) hide)
     )
@@
     )
     (path "/61d4e7b2-92e9-40a1-800c-070039f9c47a"
-      (reference "J1") (unit 1) (value "Conn_Coaxial") (footprint "Connector_Coaxial:SMA_Amphenol_132134-10_Vertical")
+      (reference "J1") (unit 1) (value "Conn_Coaxial") (footprint "Connector_Coaxial:SMA_Amphenol_132289_EdgeMount")
     )
     (path "/ac556117-03f8-4778-a611-923dc8fe4ce3"
-      (reference "J2") (unit 1) (value "Conn_Coaxial") (footprint "Connector_Coaxial:SMA_Amphenol_132134-10_Vertical")
+      (reference "J2") (unit 1) (value "Conn_Coaxial") (footprint "Connector_Coaxial:SMA_Amphenol_132289_EdgeMount")
     )
     (path "/ca4e2343-5699-4048-8586-f5d58d3345ef"
@@
     )
     (path "/85623dad-fcd9-4cfe-9f60-5be992a5a028"
-      (reference "J4") (unit 1) (value "Conn_Coaxial") (footprint "Connector_Coaxial:SMA_Amphenol_132134-10_Vertical")
+      (reference "J4") (unit 1) (value "Conn_Coaxial") (footprint "Connector_Coaxial:SMA_Amphenol_132289_EdgeMount")
     )
     (path "/60517113-5ce8-4643-acdd-1dc307a01e8a"

Commit message: Update Footprint for PAM-42 and update pcb layout to use it
Parts:
- M1: footprint Library:PAM42 -> Library:PAM42-Solder
Changed lines of the file:
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@@
       (effects (font (size 1.27 1.27)) (justify right))
     )
-    (property "Footprint" "Library:PAM42" (id 2) (at 160.02 62.23 0)
+    (property "Footprint" "Library:PAM42-Solder" (id 2) (at 160.02 62.23 0)
       (effects (font (size 1.27 1.27)) hide)
     )
@@
     )
     (path "/e7774fcd-cb69-41c1-9cd0-fa9aa054407e"
-      (reference "M1") (unit 1) (value "PAM-42") (footprint "Library:PAM42")
+      (reference "M1") (unit 1) (value "PAM-42") (footprint "Library:PAM42-Solder")
     )
     (path "/4429adbc-7361-40ed-8fb8-57433752d1a3"
