File: KiCAD/TrackingGenerator.kicad_pcb (KiCad board)
At the start: 4 copper layers, 84.4 x 60.3 mm, 65 parts, among them IC1 ABA-52563-BLKG, IC2 ABA-52563-BLKG, IC3 ABA-52563-BLKG, J1 Conn_Coaxial, J2 Conn_Coaxial, J3 Screw_Terminal_01x02, J4 Conn_Coaxial, M1 PAM-42, U1 L7805

Commit message: PCB Update
Routing:
- net Net-(M1-Pad4): track 1.73 -> 5.34 mm
